Commit message: [modify]navigation stack

File: src/2D_Navigation_Stack/urdf/wheel_robot_base.urdf.xacro (robot description, xacro)
@@ -95,7 +95,31 @@
   </gazebo>
   <!-- Hokuyo Laser scanner -->
+  <property name="hokuyo_size" value="0.1" />
+  <!-- hokuyo -->
+  <link name="laser">
+    <visual>
+      <origin xyz="0 0 0" rpy="0 0 0" />
+      <geometry>
+        <cylinder length="${hokuyo_size * 2}" radius="${hokuyo_size}" />
+      </geometry>
+      <material name="Gray" />
+    </visual>
+  </link>
+  <joint name="hokuyo_joint" type="fixed">
+    <origin xyz="${hokuyo_size/2} 0 ${0.2+hokuyo_size/4}" rpy="0 0 0" />
+    <parent link="base_link"/>
+    <child link="laser" />
+  </joint>
+  <gazebo reference="laser">
+    <material>Gazebo/Gray</material>
+    <turnGravityOff>false</turnGravityOff>
+    <sensor type="ray" name="head_hokuyo_sensor">
+      <pose>${hokuyo_size/2} 0 0 0 0 0</pose>
+    </sensor>
+  </gazebo>
+  <!-- Hokuyo Laser scanner -->
   <!-- property name="hokuyo_size" value="0.1" /> -->
   <!-- hokuyo -->
-  <!-- <link name="hokuyo_link">
+  <!-- <link name="laser">
     <visual>
       <origin xyz="0 0 0" rpy="0 0 0" />
@@ -110,7 +134,7 @@
     <origin xyz="${hokuyo_size/2} 0 ${0.2+hokuyo_size/4}" rpy="0 0 0" />
     <parent link="base_link"/>
-    <child link="hokuyo_link" />
+    <child link="laser" />
   </joint>
-  <gazebo reference="hokuyo_link">
+  <gazebo reference="laser">
     <material>Gazebo/Gray</material>
     <turnGravityOff>false</turnGravityOff>
@@ -136,5 +160,5 @@
       <plugin name="gazebo_ros_head_hokuyo_controller" filename="libgazebo_ros_laser.so">
         <topicName>/scan</topicName>
-        <frameName>hokuyo_link</frameName>
+        <frameName>laser</frameName>
       </plugin>
     </sensor>
