Commit message: [modify]param files

File: src/2D_Navigation_Stack/urdf/2WD_laser.urdf.xacro (robot description, xacro)
@@ -167,9 +167,9 @@
   <!-- SENSORS -->
   <!-- hokuyo -->
-  <link name="hokuyo_link">
+  <link name="laser">
     <visual>
       <origin xyz="0 0 0" rpy="0 0 0" />
       <geometry>
-        <box size="${hokuyo_size} ${hokuyo_size} ${hokuyo_size}"/>
+        <mesh filename="package://2D_Navigation_Stack/meshes/hokuyo.dae"/>
       </geometry>
       <material name="Blue" />
@@ -179,7 +179,7 @@
     <origin xyz="${base_radius - hokuyo_size/2} 0 ${base_height+hokuyo_size/4}" rpy="0 0 0" />
     <parent link="base_link"/>
-    <child link="hokuyo_link" />
+    <child link="laser" />
   </joint>
-  <gazebo reference="hokuyo_link">
+  <gazebo reference="laser">
     <material>Gazebo/Blue</material>
     <turnGravityOff>false</turnGravityOff>
@@ -205,5 +205,5 @@
       <plugin name="gazebo_ros_head_hokuyo_controller" filename="libgazebo_ros_laser.so">
         <topicName>/scan</topicName>
-        <frameName>hokuyo_link</frameName>
+        <frameName>laser</frameName>
       </plugin>
     </sensor>

File: src/2D_Navigation_Stack/urdf/4WD_laser.urdf.xacro (robot description, xacro)
@@ -97,11 +97,13 @@
   <property name="hokuyo_size" value="0.1" />
   <!-- hokuyo -->
-  <link name="hokuyo_link">
+  <link name="laser">
     <visual>
       <origin xyz="0 0 0" rpy="0 0 0" />
       <geometry>
+        <mesh filename="package://2D_Navigation_Stack/meshes/hokuyo.dae"/>
+      </geometry>
+      <!-- <geometry>
         <cylinder length="${hokuyo_size * 2}" radius="${hokuyo_size}" />
-        <!--<box size="${hokuyo_size} ${hokuyo_size} ${hokuyo_size}"/>-->
-      </geometry>
+      </geometry> -->
       <material name="Gray" />
     </visual>
@@ -114,12 +116,12 @@
     <origin xyz="${hokuyo_size/2} 0 ${0.2+hokuyo_size/4}" rpy="0 0 0" />
     <parent link="base_link"/>
-    <child link="hokuyo_link" />
+    <child link="laser" />
   </joint>
-  <gazebo reference="hokuyo_link">
+  <gazebo reference="laser">
     <material>Gazebo/Gray</material>
     <turnGravityOff>false</turnGravityOff>
     <sensor type="ray" name="head_hokuyo_sensor">
       <pose>${hokuyo_size/2} 0 0 0 0 0</pose>
-      <visualize>true</visualize>
+      <visualize>false</visualize>
       <update_rate>40</update_rate>
       <ray>
@@ -140,5 +142,5 @@
       <plugin name="gazebo_ros_head_hokuyo_controller" filename="libgazebo_ros_laser.so">
         <topicName>/scan</topicName>
-        <frameName>hokuyo_link</frameName>
+        <frameName>laser</frameName>
       </plugin>
     </sensor>
