Commit message: [modify]DWAで少し衝突回避成功

File: src/2D_Navigation_Stack/urdf/ck9_gazebo.xacro (robot description, xacro)
@@ -1,5 +1,5 @@
 <?xml version="1.0"?>
 <robot xmlns:xacro="http://www.ros.org/wiki/xacro" name="ck9_gazebo">
-  <xacro:include filename="$(find ck9_gazebo)/urdf/ck9_gazebo.plugins.xacro" />
+  <xacro:include filename="$(find 2D_Navigation_Stack)/urdf/ck9_gazebo.plugins.xacro" />
   <xacro:property name="base_radius" value="0.15"/>
   <xacro:property name="base_len" value="0.056"/>
@@ -55,5 +55,5 @@
       <geometry>
         <mesh
-          filename="package://ck9_gazebo/meshes/ck9.stl" />>
+          filename="package://2D_Navigation_Stack/meshes/ck9.stl" />>
       </geometry>
     <material name="white"/>
@@ -84,5 +84,5 @@
         <geometry>
          <mesh scale="0.001 0.001 0.001"
-          filename="package://ck9_gazebo/meshes/wheel.stl" />
+          filename="package://2D_Navigation_Stack/meshes/wheel.stl" />
           <!--<cylinder radius="${wheel_radius}" length="0.005"/>-->
         </geometry>
@@ -182,6 +182,7 @@
     <visual>
       <origin xyz="0.023 -0.004 -0.151" rpy="0 1.571 0" />
-      <geometry>
-        <mesh filename="package://ck9_gazebo/meshes/lidar.stl"/>
+      <!-- <origin xyz="0.023 0.015 -0.151" rpy="0 1.571 3.142" /> -->
+      <geometry>
+        <mesh filename="package://2D_Navigation_Stack/meshes/lidar.stl"/>
         <!--box size="${laser_size_x} ${laser_size_y} ${laser_size_z}"/-->
       </geometry>
@@ -203,4 +204,4 @@
     <child link="sensor_laser" />
   </joint>
-  <xacro:include filename="$(find ck9_gazebo)/urdf/ck9_gazebo.diff.plugins.xacro"/>
+  <xacro:include filename="$(find 2D_Navigation_Stack)/urdf/ck9_gazebo.diff.plugins.xacro"/>
 </robot>
